Commit message: feat(kinematics): add shared tool-frame kinematics and reconcile the TCP frame
Adds so101_nexus.kinematics, a tensor-agnostic module (NumPy and torch, no
torch import) holding the quaternion algebra, the weighted pose error, and the
damped-least-squares step both backends will share, so end-effector semantics
cannot drift between them.

ee_ik_delta_q takes the raw mj_jacSite-style Jacobian and applies the
orientation weight to its rotational rows itself. Weighted least squares scales
both sides: de-weighting only the error leaves the solver holding tool
orientation at full weight, which a five-joint arm satisfies only by barely
moving (4.63 mm median tracking error against 0.16 mm when both are scaled).

The MJCF gripperframe site and the URDF gripper_frame_link named different
physical points, 19.9 mm apart along the gripper-link x axis: upstream places
its frame at the fixed fingertip, the simulator site sits between the jaws.
Moving the site would silently shift every reward, success threshold, and
recorded dataset, so so101_new_calib.urdf gains a tcp_frame_link matching the
site exactly and upstream's frame is left alone. A regression test locks the
two models together.

File: src/so101_nexus/assets/SO101/so101_new_calib.urdf (robot description, URDF)
Before this commit: robot so101_new_calib, 8 links, 7 joints
Links:
- added link tcp_frame_link, mass 1e-9
Joints:
- added joint tcp_frame_joint: type fixed, parent gripper_link, child tcp_frame_link, origin xyz=0.012 -0.000218 -0.098127 rpy=0 3.14159265 0, axis 0 0 0
